Commit message: Controller change.

File: butler_moveit_config/config/gazebo_butler.urdf (robot description, URDF)
Before this commit: robot butler, 41 links, 40 joints
Links:
- removed link gripper_robotiq_85_base_link
- removed link gripper_robotiq_85_left_finger_link
- removed link gripper_robotiq_85_left_finger_tip_link
- removed link gripper_robotiq_85_left_inner_knuckle_link
- removed link gripper_robotiq_85_left_knuckle_link
- removed link gripper_robotiq_85_right_finger_link
- removed link gripper_robotiq_85_right_finger_tip_link
- removed link gripper_robotiq_85_right_inner_knuckle_link
- removed link gripper_robotiq_85_right_knuckle_link
- added link camera_bottom_screw_frame
- added link camera_color_frame
- added link camera_color_optical_frame
- added link camera_depth_frame
- added link camera_depth_optical_frame
- added link camera_left_ir_frame
- added link camera_left_ir_optical_frame
- added link camera_link, mass 0.564; collision box size=0.02505 0.09 0.025; visual mesh filename=package://realsense2_description/meshes/d435.dae
- added link camera_right_ir_frame
- added link camera_right_ir_optical_frame
- link body: geometry collision mesh filename=package://butler_description/meshes/body/collision/body.stl; visual mesh filename=package://butler_description/meshes/body/visual/body.obj scale=0.001 0.001 0.001
- link cover_left: geometry collision mesh filename=package://butler_description/meshes/body/visual/cover_left_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; visual mesh filename=package://butler_description/meshes/body/visual/cover_left_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
Joints:
- removed joint gripper_robotiq_85_base_joint
- removed joint gripper_robotiq_85_left_finger_joint
- removed joint gripper_robotiq_85_left_finger_tip_joint
- removed joint gripper_robotiq_85_left_inner_knuckle_joint
- removed joint gripper_robotiq_85_left_knuckle_joint
- removed joint gripper_robotiq_85_right_finger_joint
- removed joint gripper_robotiq_85_right_finger_tip_joint
- removed joint gripper_robotiq_85_right_inner_knuckle_joint
- removed joint gripper_robotiq_85_right_knuckle_joint
- added joint camera_color_joint: type fixed, parent camera_depth_frame, child camera_color_frame, origin xyz=0 0.015 0 rpy=0 0 0
- added joint camera_color_optical_joint: type fixed, parent camera_color_frame, child camera_color_optical_frame, origin xyz=0 0 0 rpy=-1.5707963267948966 0 -1.5707963267948966
- added joint camera_depth_joint: type fixed, parent camera_link, child camera_depth_frame, origin xyz=0 0 0 rpy=0 0 0
- added joint camera_depth_optical_joint: type fixed, parent camera_depth_frame, child camera_depth_optical_frame, origin xyz=0 0 0 rpy=-1.5707963267948966 0 -1.5707963267948966
- added joint camera_joint: type fixed, parent ur5_tool0, child camera_bottom_screw_frame, origin xyz=-0.000854 0 0.029708 rpy=0.0 -0.786 0
- added joint camera_left_ir_joint: type fixed, parent camera_depth_frame, child camera_left_ir_frame, origin xyz=0 0.0 0 rpy=0 0 0
- added joint camera_left_ir_optical_joint: type fixed, parent camera_left_ir_frame, child camera_left_ir_optical_frame, origin xyz=0 0 0 rpy=-1.5707963267948966 0 -1.5707963267948966
- added joint camera_link_joint: type fixed, parent camera_bottom_screw_frame, child camera_link, origin xyz=0 0.0175 0.0125 rpy=0 0 0
- added joint camera_right_ir_joint: type fixed, parent camera_depth_frame, child camera_right_ir_frame, origin xyz=0 -0.05 0 rpy=0 0 0
- added joint camera_right_ir_optical_joint: type fixed, parent camera_right_ir_frame, child camera_right_ir_optical_frame, origin xyz=0 0 0 rpy=-1.5707963267948966 0 -1.5707963267948966
- joint ur5_elbow_joint: limit lower=0.0 upper=2.93005874824808 effort=150.0 velocity=3.141592653589793 -> lower=-3.141592653589793 upper=3.141592653589793 effort=150.0 velocity=3.141592653589793
- joint ur5_shoulder_lift_joint: limit lower=-3.141592653589793 upper=0.7400196028455958 effort=150.0 velocity=3.141592653589793 -> lower=-6.283185307179586 upper=6.283185307179586 effort=150.0 velocity=3.141592653589793
- joint ur5_shoulder_pan_joint: limit lower=-3.141592653589793 upper=3.141592653589793 effort=150.0 velocity=3.141592653589793 -> lower=-6.283185307179586 upper=6.283185307179586 effort=150.0 velocity=3.141592653589793
- joint ur5_wrist_1_joint: limit lower=-3.141592653589793 upper=0.0 effort=28.0 velocity=3.141592653589793 -> lower=-6.283185307179586 upper=6.283185307179586 effort=28.0 velocity=3.141592653589793
- joint ur5_wrist_2_joint: limit lower=-3.141592653589793 upper=3.141592653589793 effort=28.0 velocity=3.141592653589793 -> lower=-6.283185307179586 upper=6.283185307179586 effort=28.0 velocity=3.141592653589793
- joint ur5_wrist_3_joint: limit lower=0.5235987755982988 upper=4.799655442984406 effort=28.0 velocity=3.141592653589793 -> lower=-6.283185307179586 upper=6.283185307179586 effort=28.0 velocity=3.141592653589793
